File: PGA2040_Carrier.kicad_pcb (KiCad board)
At the start: 2 copper layers, 438.4 x 141.4 mm, 222 parts, among them J1 Conn_01x04_Pin, J2 Conn_01x04_Pin, U2 USBLC6-2SC6

Commit message: Add files via upload
Parts:
- J1, J2: footprint Connector_JST:JST_XH_B4B-XH-A_1x04_P2.50mm_Vertical -> Connector_PinHeader_2.54mm:PinHeader_1x04_P2.54mm_Vertical
- R1, R2, R3: value Resistor -> 220R
- moved J1 0.31 mm to (38.4, 54.2), turned to 90 degrees
- moved J2 0.25 mm to (455.6, 54.2), turned to 90 degrees
Routing:
- net USB_DP: track 474.0 -> 471.3 mm
- net USB_DM: track 465.2 -> 463.5 mm
- net VBUS_USB: track 432.1 -> 433.2 mm
Other:
- board size 438.4 x 141.4 mm -> 438.3 x 140.9 mm
- board text added: "TomahawkLabs"
