File: PGA2040_Carrier.kicad_pcb (KiCad board)
At the start: 2 copper layers, 438.3 x 140.9 mm, 222 parts, among them J1 Conn_01x05_Pin, J2 Conn_01x05_Pin, U2 USBLC6-2SC6

Commit message: Add files via upload
Parts:
- moved U2 22.6 mm to (441.8, 56.2), turned to 0 degrees
Routing:
- net MCU_DP: track 7.61 -> 34.9 mm
- net USB_DP: track 470.7 -> 444.6 mm
- net USB_DM: track 463.2 -> 438.4 mm
- net MCU_DM: track 10.1 -> 34.3 mm, vias 1 -> 0
- net VBUS: track 39.3 -> 46.1 mm
- net GND: track 0.00 -> 1.66 mm, vias 2 -> 3
